File: defiant.kicad_pcb (KiCad board)
At the start: 2 copper layers, 126.6 x 99.2 mm, 55 parts, among them J1 Conn_01x02_Pin, SW1 SW_Push, SW2 SW_Push, SW3 SW_DP3T, T0 SW_PUSH, T1 SW_PUSH, T2 SW_PUSH, T3 SW_PUSH, T4 SW_PUSH, U1 Seeed Studio XIAO BLE

Commit message: Update thumb keycaps to not collide with standard keycaps
Parts:
- U1: footprint Seeedstudio XIAO:XIAO-nRF52840-Sense-14P-2.54-21X17.8MM_NoLED_Handsolder -> Seeedstudio XIAO:XIAO-nRF52840-Sense-14P-2.54-21X17.8MM_Reduced_Pins
